File: hardware/gps-v3.kicad_pcb (KiCad board)
At the start: 2 copper layers, 40 x 40 mm, 38 parts, among them P1 Debug, P101 CON-SENSOR, P103 Boot, P104 U.FL, Q1 2N7002, U1 PA1616D, U101 XMC1302-32, U103 DRILL, U104 DRILL, U105 DRILL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

Commit message: prototype
Parts:
- added Fiducial_Mark: VAL**, kicad-libraries:Fiducial_Mark, F.Cu at (137.0, 132.0)
- added Fiducial_Mark: VAL**, kicad-libraries:Fiducial_Mark, F.Cu at (127.0, 113.0)
- added Fiducial_Mark: VAL**, kicad-libraries:Fiducial_Mark, F.Cu at (104.0, 107.0)
Changed lines of the file:
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@@
-(kicad_pcb (version 20171130) (host pcbnew 5.1.6-c6e7f7d~87~ubuntu20.04.1)
+(kicad_pcb (version 20171130) (host pcbnew 5.1.7-a382d34a8~87~ubuntu20.04.1)
   (general
     (thickness 1.6)
@@
     (tracks 307)
     (zones 0)
-    (modules 38)
+    (modules 41)
     (nets 52)
   )
@@
   )
   (setup
-    (last_trace_width 0.25)
+    (last_trace_width 0.2)
     (user_trace_width 0.25)
     (user_trace_width 0.3)
@@
     (pad_drill 0.6)
     (pad_to_mask_clearance 0)
-    (solder_mask_min_width 0.25)
     (aux_axis_origin 100 100)
     (grid_origin 100 100)
     (visible_elements FFFFFF7F)
     (pcbplotparams
-      (layerselection 0x00010_00000000)
-      (usegerberextensions false)
+      (layerselection 0x310fc_ffffffff)
+      (usegerberextensions true)
       (usegerberattributes false)
       (usegerberadvancedattributes false)
@@
       (drillshape 0)
       (scaleselection 1)
-      (outputdirectory "/tmp/"))
+      (outputdirectory "../../../Schreibtisch/proto/gps-v3/"))
   )
   (net 0 "")
@@
     (add_net VCC)
   )
+  (module kicad-libraries:Fiducial_Mark (layer F.Cu)
+    (at 137 132)
+    (attr smd)
+    (fp_text reference Fiducial_Mark (at 0 0) (layer F.SilkS) hide
+      (effects (font (size 0.127 0.127) (thickness 0.03302)))
+    )
+    (fp_text value VAL** (at 0 -0.29972) (layer F.SilkS) hide
+      (effects (font (size 0.127 0.127) (thickness 0.03302)))
+    )
+    (fp_circle (center 0 0) (end 1.15062 0) (layer Dwgs.User) (width 0.01016))
+    (pad 1 smd circle (at 0 0) (size 1.00076 1.00076) (layers F.Cu F.Paste F.Mask)
+      (clearance 0.65024))
+  )
+  (module kicad-libraries:Fiducial_Mark (layer F.Cu)
+    (at 127 113)
+    (attr smd)
+    (fp_text reference Fiducial_Mark (at 0 0) (layer F.SilkS) hide
+      (effects (font (size 0.127 0.127) (thickness 0.03302)))
+    )
+    (fp_text value VAL** (at 0 -0.29972) (layer F.SilkS) hide
+      (effects (font (size 0.127 0.127) (thickness 0.03302)))
+    )
+    (fp_circle (center 0 0) (end 1.15062 0) (layer Dwgs.User) (width 0.01016))
+    (pad 1 smd circle (at 0 0) (size 1.00076 1.00076) (layers F.Cu F.Paste F.Mask)
+      (clearance 0.65024))
+  )
+  (module kicad-libraries:Fiducial_Mark (layer F.Cu)
+    (at 104 107)
+    (attr smd)
+    (fp_text reference Fiducial_Mark (at 0 0) (layer F.SilkS) hide
+      (effects (font (size 0.127 0.127) (thickness 0.03302)))
+    )
+    (fp_text value VAL** (at 0 -0.29972) (layer F.SilkS) hide
+      (effects (font (size 0.127 0.127) (thickness 0.03302)))
+    )
+    (fp_circle (center 0 0) (end 1.15062 0) (layer Dwgs.User) (width 0.01016))
+    (pad 1 smd circle (at 0 0) (size 1.00076 1.00076) (layers F.Cu F.Paste F.Mask)
+      (clearance 0.65024))
+  )
   (module kicad-libraries:R0603F (layer F.Cu)

Commit message: changed resistor value
Parts:
- RP1: value 220 -> 82
Changed lines of the file:
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@@
-(kicad_pcb (version 20171130) (host pcbnew 5.1.7-a382d34a8~87~ubuntu20.04.1)
+(kicad_pcb (version 20171130) (host pcbnew "(5.1.4)-1")
   (general
     (thickness 1.6)
@@
     (aux_axis_origin 100 100)
     (grid_origin 100 100)
-    (visible_elements FFFFFF7F)
+    (visible_elements 7FFFFFFF)
     (pcbplotparams
       (layerselection 0x310fc_ffffffff)
@@
       (effects (font (size 0.2 0.2) (thickness 0.05)))
     )
-    (fp_text value 220 (at -0.025 -0.45 90) (layer F.Fab)
-      (effects (font (size 0.2 0.2) (thickness 0.05)))
-    )
+    (fp_text value 82 (at -0.025 -0.45 90) (layer F.Fab)
+      (effects (font (size 0.2 0.2) (thickness 0.05)))
+    )

Commit message: bugfix: change n ch mosfet with p ch mosfet
Parts:
- Q1: value 2N7002 -> NTR2101PT1G
- R5: value 10k -> DNP

Commit message: make power boost circuitry as DNP
Parts:
- C5, C6: value 1uF -> DNP
- L2: value 33nH -> DNP
- L3: value FB -> DNP
- Q1: value NTR2101PT1G -> DNP
- R4: value 1k -> DNP
